File: hubs/usb-demo-4/usb-demo-4.kicad_pcb (KiCad board)
At the start: 4 copper layers, 20 x 106 mm, 34 parts, among them J1 Conn_02x06_Odd_Even, J2 Conn_02x06_Odd_Even, J3 Conn_02x06_Odd_Even, J4 Conn_02x06_Odd_Even, J5 Conn_02x06_Odd_Even, U3 mini-560, Y1 Crystal_GND24

Commit message: Fix missing CC resistors on the usb-demo-4 data port
Parts:
- added R10: 5.1K, Resistor_SMD:R_0603_1608Metric, F.Cu at (128.0, 102.8)
- added R9: 5.1K, Resistor_SMD:R_0603_1608Metric, F.Cu at (112.0, 102.8)
Connections:
- USB1 pad A5: /CC1-DAT -> Net-(USB1-CC1)
- USB1 pad B5: /CC2-DAT -> Net-(USB1-CC2)
Routing:
- net Net-(USB1-CC2): track 0.00 -> 10.9 mm
- net Net-(USB1-CC1): track 0.00 -> 10.5 mm
- net GND: track 36.5 -> 39.3 mm, vias 15 -> 17
