File: hubs/usb-demo-4/usb-demo-4.kicad_sch (KiCad schematic)
At the start: 34 parts, among them J1 Conn_02x06_Odd_Even, J2 Conn_02x06_Odd_Even, J3 Conn_02x06_Odd_Even, J4 Conn_02x06_Odd_Even, J5 Conn_02x06_Odd_Even, U3 mini-560, Y1 Crystal_GND24

Commit message: Fix missing CC resistors on the usb-demo-4 data port
Parts:
- added R10, R9: 5.1K, Resistor_SMD:R_0603_1608Metric, symbol Device:R
Connections:
- net GND: now also R10.2, R9.1
- net CC1-DAT: no longer names the net of USB1.A5 (CC1)
- net CC1-DAT: now also R9.2
- net CC2-DAT: no longer names the net of USB1.B5 (CC2)
- net CC2-DAT: now also R10.1
